File: hardware/kicad/SiC_PSFB_3kW.kicad_pcb (KiCad board)
At the start: 4 copper layers, 260 x 200 mm, 157 parts, among them J1 VIN+, J2 VIN-, J3 VOUT+, J4 VOUT-, J5 +12V AUX, J6 SIGNAL, J7 NTC, Q1 C3M0060065K, Q2 C3M0060065K, Q3 C3M0060065K, Q4 C3M0060065K, Q5 IPP110N20N3 G, Q6 IPP110N20N3 G, Q7 IPP110N20N3 G, Q8 IPP110N20N3 G, T1 ETD59 18:3:3, U1 UCC28951PW, U2 UCC21520DW, U3 UCC21520DW, U4 UCC27524D

Commit message: DAB 6.6 kW platform: models, design, simulations, control+firmware (SIL), schematic, PCB generator, thermal/EMI/safety, optimisation, BOM, manufacturing, verification, report, test plan; PSFB generator refactored to BoardGen with negotiated router
Co-Authored-By: Claude Fable 5.1 <noreply@anthropic.com>
Claude-Session: https://claude.ai/code/session_01TJ4PYx4qhHYB2ApeFHUZoW
Parts:
- moved TP7 47.6 mm to (221.0, 16.0)
- moved TP6 42.1 mm to (221.0, 10.0)
- moved TP8 12.0 mm to (221.0, 22.0)
- moved TP9 10.8 mm to (221.0, 52.0)
- moved C52 8.00 mm to (201.0, 10.0)
- moved C53 8.00 mm to (206.0, 10.0)
- moved C54 8.00 mm to (211.0, 10.0)
- moved C55 8.00 mm to (201.0, 16.0)
- moved C56 8.00 mm to (201.0, 22.0)
- moved C57 8.00 mm to (206.0, 22.0)
- moved C58 8.00 mm to (211.0, 22.0)
- moved R40 8.00 mm to (196.0, 10.0)
- moved R41 8.00 mm to (216.0, 10.0)
- moved R42 8.00 mm to (196.0, 16.0)
- moved R43 8.00 mm to (206.0, 16.0)
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Routing:
- net +12V: track 398.3 -> 0.00 mm, vias 8 -> 0
- net VDD_Q1: track 219.2 -> 0.00 mm, vias 9 -> 0
- net SR_A: track 209.8 -> 0.00 mm, vias 2 -> 0
- net VREF: track 206.2 -> 0.00 mm, vias 4 -> 0
- net VEE_Q1: track 202.4 -> 0.00 mm, vias 4 -> 0
- net OUTC: track 183.8 -> 0.00 mm, vias 4 -> 0
- net OUTD: track 176.0 -> 0.00 mm, vias 4 -> 0
- net VDD_Q2: track 163.9 -> 0.00 mm, vias 6 -> 0
- net COMP: track 157.3 -> 0.00 mm, vias 3 -> 0
- net OUTB: track 156.7 -> 0.00 mm, vias 2 -> 0
- net OUTA: track 147.3 -> 0.00 mm, vias 4 -> 0
- net SS_EN: track 146.4 -> 0.00 mm, vias 3 -> 0
- net GD_Q1: track 133.9 -> 0.00 mm, vias 4 -> 0
- net SYNC: track 131.9 -> 0.00 mm, vias 1 -> 0
- net KS_Q1: track 130.2 -> 0.00 mm, vias 1 -> 0
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