File: hardware/kicad/SiC_PSFB_3kW.kicad_pcb (KiCad board)
At the start: 4 copper layers, 260 x 200 mm, 157 parts, among them J1 VIN+, J2 VIN-, J3 VOUT+, J4 VOUT-, J5 +12V AUX, J6 SIGNAL, J7 NTC, Q1 C3M0060065K, Q2 C3M0060065K, Q3 C3M0060065K, Q4 C3M0060065K, Q5 IPP110N20N3 G, Q6 IPP110N20N3 G, Q7 IPP110N20N3 G, Q8 IPP110N20N3 G, T1 ETD59 18:3:3, U1 UCC28951PW, U2 UCC21520DW, U3 UCC21520DW, U4 UCC27524D

Commit message: PSFB board: fully routed, KiCad DRC 0 errors / 0 unconnected (40 silkscreen warnings); reference placement from footprint bbox, SIP-7 silk split at the slot
Co-Authored-By: Claude Fable 5.1 <noreply@anthropic.com>
Claude-Session: https://claude.ai/code/session_01TJ4PYx4qhHYB2ApeFHUZoW
Parts:
- C1, C2, C3, C4: footprint C_Film_P37.5 -> SiC_PSFB:C_Film_P37.5
- C10, C32, C33, C37, C38, C42, C43, C47, C48, C52, C61, C9: footprint C_1206 -> SiC_PSFB:C_1206
- C11, C12, C13, C14, C15, C16: footprint C_Radial_D16_P7.5 -> SiC_PSFB:C_Radial_D16_P7.5
- C17, C18, C19, C20, C21, C22: footprint C_1210 -> SiC_PSFB:C_1210
- C30, C31, C34, C36, C39, C41, C44, C46, C49, C51, C53, C54, C55, C56, C57, C58, C59, C60, C65: footprint C_0603 -> SiC_PSFB:C_0603
- C35, C40, C45, C50: footprint C_0805 -> SiC_PSFB:C_0805
- C5, C6: footprint C_2220 -> SiC_PSFB:C_2220
- C64: footprint C_Radial_D8_P3.5 -> SiC_PSFB:C_Radial_D8_P3.5
- C7, C8: footprint C_Film_P22.5 -> SiC_PSFB:C_Film_P22.5
- CT1: footprint CT_Toroid_Straddle -> SiC_PSFB:CT_Toroid_Straddle
- CY1, CY2: footprint C_Y1_P12.5 -> SiC_PSFB:C_Y1_P12.5
- D1, D2: footprint TO-220-2_Vertical -> SiC_PSFB:TO-220-2_Vertical
- D10, D11, D12, D13, D3: footprint D_SMA -> SiC_PSFB:D_SMA
- D4, D5: footprint SOT-23 -> SiC_PSFB:SOT-23
- D6: footprint LED_0805 -> SiC_PSFB:LED_0805
- F1: footprint Fuse_6.3x32_Clips -> SiC_PSFB:Fuse_6.3x32_Clips
- H1, H2, H3, H4: footprint MountingHole_M4 -> SiC_PSFB:MountingHole_M4
- J1, J2: footprint Lug_M4 -> SiC_PSFB:Lug_M4
- J3, J4: footprint Lug_M5 -> SiC_PSFB:Lug_M5
- J5: footprint TerminalBlock_1x02_P5.08 -> SiC_PSFB:TerminalBlock_1x02_P5.08
- J6: footprint PinHeader_1x08_P2.54 -> SiC_PSFB:PinHeader_1x08_P2.54
- J7: footprint PinHeader_1x02_P2.54 -> SiC_PSFB:PinHeader_1x02_P2.54
- L1: footprint Inductor_ETD39_Lr -> SiC_PSFB:Inductor_ETD39_Lr
- L2: footprint Inductor_Toroid_D52_Lo -> SiC_PSFB:Inductor_Toroid_D52_Lo
- PS1, PS2, PS3, PS4: footprint SIP-7_IsoDCDC -> SiC_PSFB:SIP-7_IsoDCDC
- Q1, Q2, Q3, Q4: footprint TO-247-4_Vertical -> SiC_PSFB:TO-247-4_Vertical
- Q5, Q6, Q7, Q8: footprint TO-220-3_Vertical -> SiC_PSFB:TO-220-3_Vertical
- R1, R2: footprint R_2512 -> SiC_PSFB:R_2512
- R20, R21, R24, R27, R30, R33, R41, R42, R45, R46, R47, R48, R49, R50, R51, R52, R53, R54, R55, R56, R57, R58, R60, R62, R64, R66, R68, R69, R70: footprint R_0603 -> SiC_PSFB:R_0603
- R22, R23, R25, R26, R28, R29, R31, R32: footprint R_1206 -> SiC_PSFB:R_1206
- R3: footprint R_Shunt_8518 -> SiC_PSFB:R_Shunt_8518
- R40, R43, R44, R59, R61, R63, R65, R67: footprint R_0805 -> SiC_PSFB:R_0805
- T1: footprint Transformer_ETD59_PSFB -> SiC_PSFB:Transformer_ETD59_PSFB
- TP1, TP2, TP3, TP4, TP5, TP6, TP7, TP8, TP9: footprint TestPoint -> SiC_PSFB:TestPoint
- U1: footprint TSSOP-24 -> SiC_PSFB:TSSOP-24
- U2, U3: footprint SOIC-16W -> SiC_PSFB:SOIC-16W
- U4: footprint SOIC-8 -> SiC_PSFB:SOIC-8
- moved TP5 3.61 mm to (143.0, 45.0)
- moved R20 3.00 mm to (143.0, 49.0)
- moved R21 3.00 mm to (143.0, 61.0)
Routing:
- net +12V: track 0.00 -> 409.6 mm, vias 0 -> 7
- net CS: track 0.00 -> 298.3 mm, vias 0 -> 3
- net VREF: track 0.00 -> 213.7 mm, vias 0 -> 4
- net OUTC: track 0.00 -> 210.1 mm, vias 0 -> 2
- net SR_A: track 0.00 -> 197.1 mm, vias 0 -> 4
- net COMP: track 0.00 -> 186.6 mm, vias 0 -> 4
- net OUTA: track 0.00 -> 185.3 mm, vias 0 -> 2
- net OUTD: track 0.00 -> 184.5 mm, vias 0 -> 4
- net OUTB: track 0.00 -> 180.2 mm, vias 0 -> 2
- net VDD_Q1: track 0.00 -> 178.7 mm, vias 0 -> 2
- net VEE_Q1: track 0.00 -> 169.7 mm, vias 0 -> 3
- net OUTF: track 0.00 -> 149.4 mm, vias 0 -> 2
- net OUTE: track 0.00 -> 145.5 mm, vias 0 -> 4
- net SYNC: track 0.00 -> 144.9 mm, vias 0 -> 3
- net SS_EN: track 0.00 -> 143.9 mm, vias 0 -> 4
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