File: SiC_6k6_Industrial_DAB/07_KiCad_Schematics/SiC_DAB_6k6.kicad_pcb (KiCad board)
At the start: 6 copper layers, 340 x 250 mm, 261 parts, among them J1 HV+, J10 BoosterPack J1/J3, J11 BoosterPack J2/J4, J12 BoosterPack PWM, J13 +24V IN, J14 CAN, J15 UART, J16 RELAY/FAN, J17 INTERLOCK IN, J18 NTC1, J19 NTC2, J2 HV-, J20 PE, J21 PE_HV, J22 PE_LV, J3 SW_A, J4 SW_B, J5 LV+, J6 LV-, J7 SW_C, J8 SW_D, J9 L1 (via CT), Q1 C3M0032120K, Q2 C3M0032120K, Q3 C3M0032120K, Q4 C3M0032120K, Q5 C3M0016120K, Q6 C3M0016120K, Q7 C3M0016120K, Q8 C3M0016120K, U1 UCC21520DW, U10 LM393, U11 LM393, U12 74HC32, U13 TSR 3-24120, U14 TSR 1-2450, U15 AMS1117-3.3, U16 TCAN332, U17 ULN2003A, U18 PC817, U19 PC817, U2 UCC21520DW, U3 UCC21520DW, U4 UCC21520DW, U5 AMC1301, U6 AMC1301, U7 AMC1301, U8 TLV9062, U9 TLV9062

Commit message: Router: region re-route round in the hard pass, ROUTER_RESUME replay of a dumped negotiation state; DAB board run 21 intermediate files
Co-Authored-By: Claude Fable 5.1 <noreply@anthropic.com>
Claude-Session: https://claude.ai/code/session_01TJ4PYx4qhHYB2ApeFHUZoW
Routing:
- net GND: track 0.00 -> 495.1 mm, vias 0 -> 75
- net PROT_DIS: track 0.00 -> 418.4 mm, vias 0 -> 15
- net +12V: track 0.00 -> 377.5 mm, vias 0 -> 4
- net +24V: track 0.00 -> 262.6 mm, vias 0 -> 7
- net +3V3: track 0.00 -> 256.3 mm, vias 0 -> 4
- net VEE_Q8: track 0.00 -> 216.2 mm, vias 0 -> 4
- net V1_SE: track 0.00 -> 197.4 mm, vias 0 -> 5
- net KS_Q8: track 0.00 -> 193.8 mm, vias 0 -> 1
- net PE_HV: track 0.00 -> 188.2 mm
- net PWM3A: track 0.00 -> 186.7 mm, vias 0 -> 1
- net VDD_Q1: track 0.00 -> 186.2 mm, vias 0 -> 7
- net PWM2B: track 0.00 -> 184.7 mm, vias 0 -> 6
- net V2_SE: track 0.00 -> 183.9 mm, vias 0 -> 6
- net PWM3B: track 0.00 -> 177.4 mm, vias 0 -> 1
- net VDD_Q8: track 0.00 -> 176.2 mm, vias 0 -> 3
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
Commit message: DAB board: intermediate generated board files (run 22 in progress)
Co-Authored-By: Claude Fable 5.1 <noreply@anthropic.com>
Claude-Session: https://claude.ai/code/session_01TJ4PYx4qhHYB2ApeFHUZoW
Parts:
- moved U12 26.0 mm to (186.0, 44.0)
- moved J17 4.00 mm to (136.0, 160.0)
- moved U10 4.00 mm to (172.0, 62.0)
- moved U11 4.00 mm to (172.0, 80.0)
Routing:
- net GND: track 495.1 -> 0.00 mm, vias 75 -> 0
- net PROT_DIS: track 418.4 -> 0.00 mm, vias 15 -> 0
- net +12V: track 377.5 -> 0.00 mm, vias 4 -> 0
- net +24V: track 262.6 -> 0.00 mm, vias 7 -> 0
- net +3V3: track 256.3 -> 0.00 mm, vias 4 -> 0
- net VEE_Q8: track 216.2 -> 0.00 mm, vias 4 -> 0
- net V1_SE: track 197.4 -> 0.00 mm, vias 5 -> 0
- net KS_Q8: track 193.8 -> 0.00 mm, vias 1 -> 0
- net PE_HV: track 188.2 -> 0.00 mm
- net PWM3A: track 186.7 -> 0.00 mm, vias 1 -> 0
- net VDD_Q1: track 186.2 -> 0.00 mm, vias 7 -> 0
- net PWM2B: track 184.7 -> 0.00 mm, vias 6 -> 0
- net V2_SE: track 183.9 -> 0.00 mm, vias 6 -> 0
- net PWM3B: track 177.4 -> 0.00 mm, vias 1 -> 0
- net VDD_Q8: track 176.2 -> 0.00 mm, vias 3 -> 0
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