File: SiC_6k6_Industrial_DAB/07_KiCad_Schematics/hv_bridge.kicad_sch (KiCad schematic)
At the start: 26 parts, among them J1 HV+, J2 HV-, J3 SW_A, J4 SW_B, Q1 C3M0032120K, Q2 C3M0032120K, Q3 C3M0032120K, Q4 C3M0032120K

Commit message: Router: recursive rip-up retry with state snapshots, same-net task merge; DAB: per-region PE lugs with PE clearance class, net-class fixes (SW_A_CT, SH_N, SH_NS), placement fixes (U15, U18/U19, TP1, bias caps); tools/kicad README
Co-Authored-By: Claude Fable 5.1 <noreply@anthropic.com>
Claude-Session: https://claude.ai/code/session_01TJ4PYx4qhHYB2ApeFHUZoW
Parts:
- added J21: PE_HV, SiC_DAB:Lug_M5, symbol SiC_DAB:LUG
Connections:
- net PE renamed PE_HV
- net PE_HV: now also J21.1
Changed lines of the file:
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@@
   (wire (pts (xy 248.92 46.99) (xy 248.92 49.53)) (stroke (width 0) (type default))
   )
-  (global_label "PE" (shape passive) (at 248.92 49.53 270) (fields_autoplaced)
+  (global_label "PE_HV" (shape passive) (at 248.92 49.53 270) (fields_autoplaced)
     (effects (font (size 1.27 1.27)) (justify right))
     (property "Intersheetrefs" "${INTERSHEET_REFS}" (at 248.92 49.53 0) (effects (font (size 1.27 1.27)) hide))
@@
   (wire (pts (xy 269.24 46.99) (xy 269.24 49.53)) (stroke (width 0) (type default))
   )
-  (global_label "PE" (shape passive) (at 269.24 49.53 270) (fields_autoplaced)
+  (global_label "PE_HV" (shape passive) (at 269.24 49.53 270) (fields_autoplaced)
     (effects (font (size 1.27 1.27)) (justify right))
     (property "Intersheetrefs" "${INTERSHEET_REFS}" (at 269.24 49.53 0) (effects (font (size 1.27 1.27)) hide))
   )
+  (symbol (lib_id "SiC_DAB:LUG") (at 289.56 39.37 0) (unit 1)
+    (in_bom yes) (on_board yes) (dnp no)
+    (property "Reference" "J21" (at 292.1 40.64 0) (effects (font (size 1.27 1.27)) (justify left)))
+    (property "Value" "PE_HV" (at 292.1 43.18 0) (effects (font (size 1.27 1.27)) (justify left)))
+    (property "Footprint" "SiC_DAB:Lug_M5" (at 289.56 39.37 0) (effects (font (size 1.27 1.27)) (justify left) hide))
+    (property "Datasheet" "" (at 289.56 39.37 0) (effects (font (size 1.27 1.27)) (justify left) hide))
+    (property "MPN" "" (at 289.56 39.37 0) (effects (font (size 1.27 1.27)) (justify left) hide))
+    (property "Description" "PE lug of the HV region: Y-capacitor return, bonded to the HV heatsink / enclosure (the three PE lugs are joined through the chassis, not on the PCB, because no copper may cross the isolation barriers)" (at 289.56 39.37 0) (effects (font (size 1.27 1.27)) (justify left) hide))
+    (pin "1")
+    (instances (project "SiC_DAB_6k6" (path "/310d9c14-d5df-4b2b-99fc-78c5607a358c/f0cf1caa-0897-4faf-8cd7-cf2b8846ce2e" (reference "J21") (unit 1))))
+  )
+  (wire (pts (xy 289.56 36.83) (xy 289.56 34.29)) (stroke (width 0) (type default))
+  )
+  (global_label "PE_HV" (shape passive) (at 289.56 34.29 90) (fields_autoplaced)
+    (effects (font (size 1.27 1.27)) (justify left))
+    (property "Intersheetrefs" "${INTERSHEET_REFS}" (at 289.56 34.29 0) (effects (font (size 1.27 1.27)) hide))
+  )
   (symbol (lib_id "SiC_DAB:Q_NMOS_KELVIN") (at 38.1 82.55 0) (unit 1)
