File: SiC_6k6_Industrial_DAB/07_KiCad_Schematics/lv_bridge.kicad_sch (KiCad schematic)
At the start: 25 parts, among them J5 LV+, J6 LV-, J7 SW_C, J8 SW_D, Q5 C3M0016120K, Q6 C3M0016120K, Q7 C3M0016120K, Q8 C3M0016120K

Commit message: Router: recursive rip-up retry with state snapshots, same-net task merge; DAB: per-region PE lugs with PE clearance class, net-class fixes (SW_A_CT, SH_N, SH_NS), placement fixes (U15, U18/U19, TP1, bias caps); tools/kicad README
Co-Authored-By: Claude Fable 5.1 <noreply@anthropic.com>
Claude-Session: https://claude.ai/code/session_01TJ4PYx4qhHYB2ApeFHUZoW
Parts:
- added J22: PE_LV, SiC_DAB:Lug_M5, symbol SiC_DAB:LUG
Connections:
- net PE renamed PE_LV
- net PE_LV: now also J22.1
Changed lines of the file:
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@@
   (wire (pts (xy 208.28 46.99) (xy 208.28 49.53)) (stroke (width 0) (type default))
   )
-  (global_label "PE" (shape passive) (at 208.28 49.53 270) (fields_autoplaced)
+  (global_label "PE_LV" (shape passive) (at 208.28 49.53 270) (fields_autoplaced)
     (effects (font (size 1.27 1.27)) (justify right))
     (property "Intersheetrefs" "${INTERSHEET_REFS}" (at 208.28 49.53 0) (effects (font (size 1.27 1.27)) hide))
@@
   (wire (pts (xy 228.6 46.99) (xy 228.6 49.53)) (stroke (width 0) (type default))
   )
-  (global_label "PE" (shape passive) (at 228.6 49.53 270) (fields_autoplaced)
+  (global_label "PE_LV" (shape passive) (at 228.6 49.53 270) (fields_autoplaced)
     (effects (font (size 1.27 1.27)) (justify right))
     (property "Intersheetrefs" "${INTERSHEET_REFS}" (at 228.6 49.53 0) (effects (font (size 1.27 1.27)) hide))
   )
-  (symbol (lib_id "SiC_DAB:R") (at 248.92 44.45 0) (unit 1)
+  (symbol (lib_id "SiC_DAB:LUG") (at 248.92 39.37 0) (unit 1)
     (in_bom yes) (on_board yes) (dnp no)
-    (property "Reference" "R7" (at 251.46 43.18 0) (effects (font (size 1.27 1.27)) (justify left)))
-    (property "Value" "1mR" (at 251.46 45.72 0) (effects (font (size 1.27 1.27)) (justify left)))
-    (property "Footprint" "SiC_DAB:R_Shunt_8518" (at 248.92 44.45 0) (effects (font (size 1.27 1.27)) (justify left) hide))
-    (property "Datasheet" "" (at 248.92 44.45 0) (effects (font (size 1.27 1.27)) (justify left) hide))
-    (property "MPN" "Vishay WSBS8518L1000JK" (at 248.92 44.45 0) (effects (font (size 1.27 1.27)) (justify left) hide))
-    (property "Description" "LV port current shunt 1 mOhm (33 A -> 33 mV)" (at 248.92 44.45 0) (effects (font (size 1.27 1.27)) (justify left) hide))
+    (property "Reference" "J22" (at 251.46 40.64 0) (effects (font (size 1.27 1.27)) (justify left)))
+    (property "Value" "PE_LV" (at 251.46 43.18 0) (effects (font (size 1.27 1.27)) (justify left)))
+    (property "Footprint" "SiC_DAB:Lug_M5" (at 248.92 39.37 0) (effects (font (size 1.27 1.27)) (justify left) hide))
+    (property "Datasheet" "" (at 248.92 39.37 0) (effects (font (size 1.27 1.27)) (justify left) hide))
+    (property "MPN" "" (at 248.92 39.37 0) (effects (font (size 1.27 1.27)) (justify left) hide))
+    (property "Description" "PE lug of the LV region: Y-capacitor return, bonded to the LV heatsink / enclosure" (at 248.92 39.37 0) (effects (font (size 1.27 1.27)) (justify left) hide))
+    (pin "1")
+    (instances (project "SiC_DAB_6k6" (path "/310d9c14-d5df-4b2b-99fc-78c5607a358c/cd16e722-41dd-4b3a-96da-4aebe98b0a5d" (reference "J22") (unit 1))))
+  )
+  (wire (pts (xy 248.92 36.83) (xy 248.92 34.29)) (stroke (width 0) (type default))
+  )
+  (global_label "PE_LV" (shape passive) (at 248.92 34.29 90) (fields_autoplaced)
+    (effects (font (size 1.27 1.27)) (justify left))
+    (property "Intersheetrefs" "${INTERSHEET_REFS}" (at 248.92 34.29 0) (effects (font (size 1.27 1.27)) hide))
+  )
+  (symbol (lib_id "SiC_DAB:R") (at 269.24 44.45 0) (unit 1)
+    (in_bom yes) (on_board yes) (dnp no)
+    (property "Reference" "R7" (at 271.78 43.18 0) (effects (font (size 1.27 1.27)) (justify left)))
+    (property "Value" "1mR" (at 271.78 45.72 0) (effects (font (size 1.27 1.27)) (justify left)))
+    (property "Footprint" "SiC_DAB:R_Shunt_8518" (at 269.24 44.45 0) (effects (font (size 1.27 1.27)) (justify left) hide))
+    (property "Datasheet" "" (at 269.24 44.45 0) (effects (font (size 1.27 1.27)) (justify left) hide))
+    (property "MPN" "Vishay WSBS8518L1000JK" (at 269.24 44.45 0) (effects (font (size 1.27 1.27)) (justify left) hide))
+    (property "Description" "LV port current shunt 1 mOhm (33 A -> 33 mV)" (at 269.24 44.45 0) (effects (font (size 1.27 1.27)) (justify left) hide))
     (pin "1")
     (pin "2")
     (instances (project "SiC_DAB_6k6" (path "/310d9c14-d5df-4b2b-99fc-78c5607a358c/cd16e722-41dd-4b3a-96da-4aebe98b0a5d" (reference "R7") (unit 1))))
   )
-  (wire (pts (xy 248.92 39.37) (xy 248.92 36.83)) (stroke (width 0) (type default))
+  (wire (pts (xy 269.24 39.37) (xy 269.24 36.83)) (stroke (width 0) (type default))
   )
-  (global_label "LV_N" (shape passive) (at 248.92 36.83 90) (fields_autoplaced)
+  (global_label "LV_N" (shape passive) (at 269.24 36.83 90) (fields_autoplaced)
     (effects (font (size 1.27 1.27)) (justify left))
-    (property "Intersheetrefs" "${INTERSHEET_REFS}" (at 248.92 36.83 0) (effects (font (size 1.27 1.27)) hide))
+    (property "Intersheetrefs" "${INTERSHEET_REFS}" (at 269.24 36.83 0) (effects (font (size 1.27 1.27)) hide))
   )
-  (wire (pts (xy 248.92 49.53) (xy 248.92 52.07)) (stroke (width 0) (type default))
+  (wire (pts (xy 269.24 49.53) (xy 269.24 52.07)) (stroke (width 0) (type default))
   )
-  (global_label "SH_N" (shape passive) (at 248.92 52.07 270) (fields_autoplaced)
+  (global_label "SH_N" (shape passive) (at 269.24 52.07 270) (fields_autoplaced)
     (effects (font (size 1.27 1.27)) (justify right))
-    (property "Intersheetrefs" "${INTERSHEET_REFS}" (at 248.92 52.07 0) (effects (font (size 1.27 1.27)) hide))
+    (property "Intersheetrefs" "${INTERSHEET_REFS}" (at 269.24 52.07 0) (effects (font (size 1.27 1.27)) hide))
   )
   (symbol (lib_id "SiC_DAB:Q_NMOS_KELVIN") (at 38.1 82.55 0) (unit 1)
