File: SiC_6k6_Industrial_DAB/07_KiCad_Schematics/sensing_protection.kicad_sch (KiCad schematic)
At the start: 65 parts, among them J9 L1 (via CT), U10 LM393, U11 LM393, U12 74HC32, U5 AMC1301, U6 AMC1301, U7 AMC1301, U8 TLV9062, U9 TLV9062

Commit message: Router hard pass with rip-up retry, exact halo radii, via cost dilation; DAB: driver passives off the fan-out corridors, PS9/PS10 SIP-7 1 W module footprint, 0.5 mm control-power tracks; PSFB: DT resistor/TP placement
- NegotiatedRouter: full/small halo masks give the exact d < hw_a+hw_b+clearance
  overlap test; A* via placement sees the via halo; nets still in conflict after
  the negotiation are re-routed against hard obstacles, with a bounded rip-up
  retry, so emitted copper never violates the clearance model.
- Fan-out: plane-net vias 1.2 mm beyond the long stubs; corridors long+1.5 mm;
  unreachable terminals are reported.
- plot_board.py: matplotlib region renderer for layout review.
- DAB: PS9/PS10 changed from a 2.54 mm SIP-4 (cannot meet the 5.5 mm module
  creepage rule) to a SIP-7 outline 1 W module (part TBD, flagged in BOM and
  insulation table); DT resistors / VCCI caps moved clear of the driver
  fan-out corridors; private regions and slots for PS9/PS10.

Co-Authored-By: Claude Fable 5.1 <noreply@anthropic.com>
Claude-Session: https://claude.ai/code/session_01TJ4PYx4qhHYB2ApeFHUZoW
Parts:
- PS10: value R1SE-0505 -> ISO 5V/5V 1W SIP-7; footprint SiC_DAB:SIP-4_IsoDCDC -> SiC_DAB:SIP-7_IsoDCDC_1W; MPN RECOM R1SE-0505/H -> TBD - as PS9
- PS9: value R1SE-0505 -> ISO 5V/5V 1W SIP-7; footprint SiC_DAB:SIP-4_IsoDCDC -> SiC_DAB:SIP-7_IsoDCDC_1W; MPN RECOM R1SE-0505/H (verify pinout) -> TBD - 1 W 5 V->5 V isolated module, SIP-7 outline with >= 7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
Changed lines of the file:
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@@
     (in_bom yes) (on_board yes) (dnp no)
     (property "Reference" "PS9" (at 90.17 34.29 0) (effects (font (size 1.27 1.27)) (justify left)))
-    (property "Value" "R1SE-0505" (at 90.17 44.45 0) (effects (font (size 1.27 1.27)) (justify left)))
-    (property "Footprint" "SiC_DAB:SIP-4_IsoDCDC" (at 99.06 39.37 0) (effects (font (size 1.27 1.27)) (justify left) hide))
+    (property "Value" "ISO 5V/5V 1W SIP-7" (at 90.17 44.45 0) (effects (font (size 1.27 1.27)) (justify left)))
+    (property "Footprint" "SiC_DAB:SIP-7_IsoDCDC_1W" (at 99.06 39.37 0) (effects (font (size 1.27 1.27)) (justify left) hide))
     (property "Datasheet" "" (at 99.06 39.37 0) (effects (font (size 1.27 1.27)) (justify left) hide))
-    (property "MPN" "RECOM R1SE-0505/H (verify pinout)" (at 99.06 39.37 0) (effects (font (size 1.27 1.27)) (justify left) hide))
+    (property "MPN" "TBD - 1 W 5 V->5 V isolated module, SIP-7 outline with >= 7.6 mm input/output pin gap, reinforced-rated (a 2.54 mm pitch SIP-4 such as R1SE cannot meet the 5.5 mm module creepage rule)" (at 99.06 39.37 0) (effects (font (size 1.27 1.27)) (justify left) hide))
     (property "Description" "1 W isolated 5 V for the HV-side sensor" (at 99.06 39.37 0) (effects (font (size 1.27 1.27)) (justify left) hide))
     (pin "1")
@@
     (in_bom yes) (on_board yes) (dnp no)
     (property "Reference" "PS10" (at 90.17 69.85 0) (effects (font (size 1.27 1.27)) (justify left)))
-    (property "Value" "R1SE-0505" (at 90.17 80.01 0) (effects (font (size 1.27 1.27)) (justify left)))
-    (property "Footprint" "SiC_DAB:SIP-4_IsoDCDC" (at 99.06 74.93 0) (effects (font (size 1.27 1.27)) (justify left) hide))
+    (property "Value" "ISO 5V/5V 1W SIP-7" (at 90.17 80.01 0) (effects (font (size 1.27 1.27)) (justify left)))
+    (property "Footprint" "SiC_DAB:SIP-7_IsoDCDC_1W" (at 99.06 74.93 0) (effects (font (size 1.27 1.27)) (justify left) hide))
     (property "Datasheet" "" (at 99.06 74.93 0) (effects (font (size 1.27 1.27)) (justify left) hide))
-    (property "MPN" "RECOM R1SE-0505/H" (at 99.06 74.93 0) (effects (font (size 1.27 1.27)) (justify left) hide))
+    (property "MPN" "TBD - as PS9" (at 99.06 74.93 0) (effects (font (size 1.27 1.27)) (justify left) hide))
     (property "Description" "1 W isolated 5 V for the LV-side sensors" (at 99.06 74.93 0) (effects (font (size 1.27 1.27)) (justify left) hide))
     (pin "1")
